File: hardware/kicad/kiosk.kicad_sch (KiCad schematic)
At the start: 15 parts, among them J10 Jack 5V rail 1, J11 Jack 5V rail 2, J13 PCF8574 - de cam hang P, J3 LCD 4.0in ST7796S + GT911, J4 VL53L1X, J5 PCF8574 - han day toi hang 4 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, J6 DS3231, J7 MAX98357A, J9 SG90 servo, U1 ESP32-S3-CAM N16R8

Commit message: fix(hardware): put the expander's socket and wire holes back the right way
I swapped them last commit on my own reasoning about which row holds the
module better, against what had already been decided: the four supply
pins are soldered pointing down and seat in J5; the port row stays
pointing up and takes wire, stripped and soldered into J13.

J13 keeps all nine holes even though three carry a signal. The six spare
ones cost nothing now and save cutting the board later.

J13 also moves into the gap between the panel and the module, where it
was overlapping the panel's area.
Parts:
- J13: value PCF8574 - de cam hang P -> PCF8574 - han day tu hang P; footprint Connector_PinSocket_2.54mm:PinSocket_1x09_P2.54mm_Vertical -> Connector_PinHeader_2.54mm:PinHeader_1x09_P2.54mm_Vertical
- J5: value PCF8574 - han day toi hang 4 chan -> PCF8574 - de cam 4 chan nguon; footprint Connector_PinHeader_2.54mm:PinHeader_1x04_P2.54mm_Vertical -> Connector_PinSocket_2.54mm:PinSocket_1x04_P2.54mm_Vertical
Changed lines of the file:
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@@
     (exclude_from_sim no) (in_bom yes) (on_board yes) (dnp no)
     (property "Reference" "J5" (at 190.5 133.35 0) (effects (font (size 1.27 1.27))))
-    (property "Value" "PCF8574 - han day toi hang 4 chan" (at 190.5 152.4 0) (effects (font (size 1.27 1.27))))
-    (property "Footprint" "Connector_PinHeader_2.54mm:PinHeader_1x04_P2.54mm_Vertical" (at 190.5 142.24 0)
+    (property "Value" "PCF8574 - de cam 4 chan nguon" (at 190.5 152.4 0) (effects (font (size 1.27 1.27))))
+    (property "Footprint" "Connector_PinSocket_2.54mm:PinSocket_1x04_P2.54mm_Vertical" (at 190.5 142.24 0)
       (effects (font (size 1.27 1.27)) hide))
     (property "Datasheet" "" (at 190.5 142.24 0) (effects (font (size 1.27 1.27)) hide))
@@
     (exclude_from_sim no) (in_bom yes) (on_board yes) (dnp no)
     (property "Reference" "J13" (at 190.5 157.48 0) (effects (font (size 1.27 1.27))))
-    (property "Value" "PCF8574 - de cam hang P" (at 190.5 189.23 0) (effects (font (size 1.27 1.27))))
-    (property "Footprint" "Connector_PinSocket_2.54mm:PinSocket_1x09_P2.54mm_Vertical" (at 190.5 172.72 0)
+    (property "Value" "PCF8574 - han day tu hang P" (at 190.5 189.23 0) (effects (font (size 1.27 1.27))))
+    (property "Footprint" "Connector_PinHeader_2.54mm:PinHeader_1x09_P2.54mm_Vertical" (at 190.5 172.72 0)
       (effects (font (size 1.27 1.27)) hide))
     (property "Datasheet" "" (at 190.5 172.72 0) (effects (font (size 1.27 1.27)) hide))

Commit message: feat(hardware): land the panel's microSD row as four bare holes
J14 drills the four pins the panel carries on its far edge and connects
none of them. Drilling without connecting is nearly free; not drilling is
final, because the board is printed before anyone finds out whether that
row came populated, and a pin soldered there holds the panel off its
8.5 mm standoffs and leaves the four screws bending it instead of
holding it. The holes also take a soldered wire later, which is the same
job J13 already does for the expander's port row.

They stay unconnected because SD_CS has no pin to reach: the other three
would share SPI2 with the panel itself, but section 2.4 is out of ordinary
GPIO and the only candidate is GPIO48, which costs the status LED and is
therefore a section 1.2 decision, not a routing one.

Position is assumed centred on the far edge, mirroring the header on the
near one, and clears both top mounting holes by 20 mm. A few millimetres
of error costs nothing while the holes are only a place to solder a wire.

Task: E14-T8
Parts:
- added J14: LCD microSD - lo cho, chua noi day, Connector_PinHeader_2.54mm:PinHeader_1x04_P2.54mm_Vertical, symbol kiosk:J14
Connections:
- no-connect marks 32 -> 36
Changed lines of the file:
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@@
     (effects (font (size 1.27 1.27)) (justify right bottom))
 )
+  (symbol (lib_id "kiosk:J14") (at 190.5 238.76 0) (unit 1)
+    (exclude_from_sim no) (in_bom yes) (on_board yes) (dnp no)
+    (property "Reference" "J14" (at 190.5 229.86999999999998 0) (effects (font (size 1.27 1.27))))
+    (property "Value" "LCD microSD - lo cho, chua noi day" (at 190.5 248.92 0) (effects (font (size 1.27 1.27))))
+    (property "Footprint" "Connector_PinHeader_2.54mm:PinHeader_1x04_P2.54mm_Vertical" (at 190.5 238.76 0)
+      (effects (font (size 1.27 1.27)) hide))
+    (property "Datasheet" "" (at 190.5 238.76 0) (effects (font (size 1.27 1.27)) hide))
+    (pin "1")
+    (pin "2")
+    (pin "3")
+    (pin "4")
+    (instances
+      (project "kiosk"
+        (path "/b0a1c2d3-0000-4000-8000-000000000001" (reference "J14") (unit 1))
+      )
+    )
+  )
+  (no_connect (at 175.26 234.95))
+  (no_connect (at 175.26 237.48999999999998))
+  (no_connect (at 175.26 240.03))
+  (no_connect (at 175.26 242.57))
   (symbol (lib_id "kiosk:J4") (at 190.5 93.98 0) (unit 1)
     (exclude_from_sim no) (in_bom yes) (on_board yes) (dnp no)

Commit message: fix(hardware): specify a 5 mm can for the panel's capacitor
C4 had 0.25 mm of courtyard either side — the tightest clearance on the
board, and it is there because a 6.8 mm outline was put in a 7.30 mm gap.
The gap cannot grow: it is fixed at 7.30 by balancing it against the two
on the other side of the panel, and those are bounded by the board edge on
one end and the devkit's pin names on the other.

So the can shrinks instead. A 100 uF in a 5 mm body is an ordinary part,
and the 5.0 and 6.3 mm packages share the same 2.50 mm lead pitch, so not
a single drill moves — the change is a specification of what to buy, not a
layout change. Clearance goes to 0.90 mm a side.

Buying the 6.3 mm can by mistake still fits the holes. It just sits where
it sat before this commit.

Task: E14-T8
Parts:
- C4: footprint Capacitor_THT:CP_Radial_D6.3mm_P2.50mm -> Capacitor_THT:CP_Radial_D5.0mm_P2.50mm
Changed lines of the file:
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@@
     (property "Reference" "C4" (at 345.44 187.96 0) (effects (font (size 1.27 1.27))))
     (property "Value" "100uF" (at 345.44 204.47 0) (effects (font (size 1.27 1.27))))
-    (property "Footprint" "Capacitor_THT:CP_Radial_D6.3mm_P2.50mm" (at 345.44 195.58 0)
+    (property "Footprint" "Capacitor_THT:CP_Radial_D5.0mm_P2.50mm" (at 345.44 195.58 0)
       (effects (font (size 1.27 1.27)) hide))
     (property "Datasheet" "" (at 345.44 195.58 0) (effects (font (size 1.27 1.27)) hide))
