File: hardware/kicad/kiosk.kicad_sch (KiCad schematic)
At the start: 18 parts, among them J10 Jack 5V rail 1, J11 Jack 5V rail 2, J13 PCF8574 - han day tu hang P, J14 LCD microSD - lo cho, chua no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, J16 USB-C - hai lo nguon ve rail 1, J18 microUSB - hai lo nguon ve ra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, J3 LCD 4.0in ST7796S + GT911, J4 VL53L1X, J5 PCF8574 - de cam 4 chan nguon, J6 DS3231, J7 MAX98357A, J9 SG90 servo, U1 ESP32-S3-CAM N16R8

Commit message: build(hardware): regenerate the board with the panel's regulator on it
check_schematic 0, check_pcb 0, DRC 0 violations and 0 unconnected pads.
Generating twice in a row gives byte-identical files.

Task: E7-T16
Parts:
- added C5: 470uF, Capacitor_THT:CP_Radial_D8.0mm_P3.50mm, symbol kiosk:C5
- added U2: AMS1117-3.3 - rail rieng cho LCD, Connector_PinSocket_2.54mm:PinSocket_1x03_P2.54mm_Vertical, symbol kiosk:U2
Connections:
- net +3V3: no longer C4.1, J3.1 (VCC)
- net +5V_R1: now also C5.1, U2.1 (VIN)
- net GND: now also C5.2, U2.2 (GND)
- new net +3V3_LCD: C4.1, J3.1 (VCC), U2.3 (VOUT)
Changed lines of the file:
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@@
   (wire (pts (xy 96.52000000000001 31.749999999999996) (xy 91.44000000000001 31.749999999999996))
     (stroke (width 0) (type default)))
-  (label "+3V3" (at 91.44000000000001 31.749999999999996 180)
+  (label "+3V3_LCD" (at 91.44000000000001 31.749999999999996 180)
     (effects (font (size 1.27 1.27)) (justify right bottom))
 )
@@
     (effects (font (size 1.27 1.27)) (justify right bottom))
 )
+  (symbol (lib_id "kiosk:U2") (at 181.61 250.19 0) (unit 1)
+    (exclude_from_sim no) (in_bom yes) (on_board yes) (dnp no)
+    (property "Reference" "U2" (at 181.61 242.57 0) (effects (font (size 1.27 1.27))))
+    (property "Value" "AMS1117-3.3 - rail rieng cho LCD" (at 181.61 259.08 0) (effects (font (size 1.27 1.27))))
+    (property "Footprint" "Connector_PinSocket_2.54mm:PinSocket_1x03_P2.54mm_Vertical" (at 181.61 250.19 0)
+      (effects (font (size 1.27 1.27)) hide))
+    (property "Datasheet" "" (at 181.61 250.19 0) (effects (font (size 1.27 1.27)) hide))
+    (pin "1")
+    (pin "2")
+    (pin "3")
+    (instances
+      (project "kiosk"
+        (path "/b0a1c2d3-0000-4000-8000-000000000001" (reference "U2") (unit 1))
+      )
+    )
+  )
+  (wire (pts (xy 166.37 247.65) (xy 161.29 247.65))
+    (stroke (width 0) (type default)))
+  (label "+5V_R1" (at 161.29 247.65 180)
+    (effects (font (size 1.27 1.27)) (justify right bottom))
+)
+  (wire (pts (xy 166.37 250.19) (xy 161.29 250.19))
+    (stroke (width 0) (type default)))
+  (label "GND" (at 161.29 250.19 180)
+    (effects (font (size 1.27 1.27)) (justify right bottom))
+)
+  (wire (pts (xy 166.37 252.73000000000002) (xy 161.29 252.73000000000002))
+    (stroke (width 0) (type default)))
+  (label "+3V3_LCD" (at 161.29 252.73000000000002 180)
+    (effects (font (size 1.27 1.27)) (justify right bottom))
+)
   (symbol (lib_id "kiosk:R1") (at 132.08 153.67 0) (unit 1)
     (exclude_from_sim no) (in_bom yes) (on_board yes) (dnp no)
@@
   (wire (pts (xy 132.08 43.18) (xy 137.16000000000003 43.18))
     (stroke (width 0) (type default)))
-  (label "+3V3" (at 137.16000000000003 43.18 0)
+  (label "+3V3_LCD" (at 137.16000000000003 43.18 0)
     (effects (font (size 1.27 1.27)) (justify left bottom))
 )
@@
     (effects (font (size 1.27 1.27)) (justify left bottom))
 )
+  (symbol (lib_id "kiosk:C5") (at 181.61 271.78 0) (unit 1)
+    (exclude_from_sim no) (in_bom yes) (on_board yes) (dnp no)
+    (property "Reference" "C5" (at 181.61 264.15999999999997 0) (effects (font (size 1.27 1.27))))
+    (property "Value" "470uF" (at 181.61 280.67 0) (effects (font (size 1.27 1.27))))
+    (property "Footprint" "Capacitor_THT:CP_Radial_D8.0mm_P3.50mm" (at 181.61 271.78 0)
+      (effects (font (size 1.27 1.27)) hide))
+    (property "Datasheet" "" (at 181.61 271.78 0) (effects (font (size 1.27 1.27)) hide))
+    (pin "1")
+    (pin "2")
+    (instances
+      (project "kiosk"
+        (path "/b0a1c2d3-0000-4000-8000-000000000001" (reference "C5") (unit 1))
+      )
+    )
+  )
+  (wire (pts (xy 181.61 266.7) (xy 186.69000000000003 266.7))
+    (stroke (width 0) (type default)))
+  (label "+5V_R1" (at 186.69000000000003 266.7 0)
+    (effects (font (size 1.27 1.27)) (justify left bottom))
+)
+  (wire (pts (xy 181.61 276.85999999999996) (xy 186.69000000000003 276.85999999999996))
+    (stroke (width 0) (type default)))
+  (label "GND" (at 186.69000000000003 276.85999999999996 0)
+    (effects (font (size 1.27 1.27)) (justify left bottom))
+)
